Commit message: Recentrer l'axe de rotation des roues au niveau du sol et simplifier la collision en sphère
Le joint continuous tournait autour du moyeu moteur (8,2 cm du sol) alors
que le contact réel se fait au niveau des roues folles (2,0 cm), ce qui
aurait produit une orbite plutôt qu'un roulement dans Gazebo. L'origine du
joint est déplacée à la hauteur des roues folles, tous les visuels sont
compensés en Z pour garder le rendu RViz identique, et la collision boîte
est remplacée par une sphère pour un contact ponctuel avec le sol.

File: src/robot_devastator_description/urdf/roues.xacro (robot description, xacro)
@@ -32,5 +32,5 @@
           <cylinder radius="${rayon_roue}" length="${largeur_roue}"/>
         </geometry>
-        <origin xyz="0 0 0" rpy="${pi/2} 0 0"/>
+        <origin xyz="0 0 ${-z_folle}" rpy="${pi/2} 0 0"/>
         <material name="noir"/>
       </visual>
@@ -39,5 +39,5 @@
           <cylinder radius="${rayon_roue}" length="${largeur_roue}"/>
         </geometry>
-        <origin xyz="-${empattement_arriere} 0 ${z_folle}" rpy="${pi/2} 0 0"/>
+        <origin xyz="-${empattement_arriere} 0 0" rpy="${pi/2} 0 0"/>
         <material name="argent"/>
       </visual>
@@ -46,5 +46,5 @@
           <cylinder radius="${rayon_roue}" length="${largeur_roue}"/>
         </geometry>
-        <origin xyz="${empattement_avant} 0 ${z_folle}" rpy="${pi/2} 0 0"/>
+        <origin xyz="${empattement_avant} 0 0" rpy="${pi/2} 0 0"/>
         <material name="argent"/>
       </visual>
@@ -53,5 +53,5 @@
           <box size="0.1012 ${largeur_roue} ${2*rayon_roue}"/>
         </geometry>
-        <origin xyz="-0.040 0 ${z_folle/2}" rpy="0 2.4826 0"/>
+        <origin xyz="-0.040 0 ${-z_folle/2}" rpy="0 2.4826 0"/>
         <material name="orange"/>
       </visual>
@@ -60,5 +60,5 @@
           <box size="0.1422 ${largeur_roue} ${2*rayon_roue}"/>
         </geometry>
-        <origin xyz="0.064 0 ${z_folle/2}" rpy="0 0.4512 0"/>
+        <origin xyz="0.064 0 ${-z_folle/2}" rpy="0 0.4512 0"/>
         <material name="noir"/>
       </visual>
@@ -67,12 +67,12 @@
           <box size="0.208 ${largeur_roue} ${2*rayon_roue}"/>
         </geometry>
-        <origin xyz="0.024 0 ${z_folle}" rpy="0 0 0"/>
+        <origin xyz="0.024 0 0" rpy="0 0 0"/>
         <material name="noir"/>
       </visual>
       <collision>
         <geometry>
-          <box size="${empattement_arriere+empattement_avant+2*rayon_roue} ${largeur_roue} ${2*rayon_roue}"/>
+          <sphere radius="${rayon_roue}"/>
         </geometry>
-        <origin xyz="${(empattement_avant-empattement_arriere)/2} 0 ${z_folle}" rpy="0 0 0"/>
+        <origin xyz="0 0 0" rpy="0 0 0"/>
       </collision>
       <inertial>
@@ -84,5 +84,5 @@
       <parent link="base_link"/>
       <child  link="${nom}_wheel"/>
-      <origin xyz="0 ${y_signe * y_roue} 0" rpy="0 0 0"/>
+      <origin xyz="0 ${y_signe * y_roue} ${z_folle}" rpy="0 0 0"/>
       <axis xyz="0 1 0"/>
     </joint>

Commit message: Correctif URDF

File: src/robot_devastator_description/urdf/roues.xacro (robot description, xacro)
@@ -22,15 +22,15 @@
     <color rgba="0.1 0.1 0.1 1.0"/>
   </material>
-  <!-- Macro réutilisable pour une roue -->
+  <!-- Macro du visuel statique d'une chenille (fixed, ne bouge jamais) -->
   <!-- La rotation de π/2 autour de X oriente les cylindres sur l'axe Y -->
   <!-- La géométrie visuelle forme une chenille triangulaire : roue menante + 2 roues -->
   <!-- folles, reliées par 3 boîtes formant le contour (dont le brin horizontal au sol) -->
-  <xacro:macro name="roue" params="nom y_signe">
-    <link name="${nom}_wheel">
+  <xacro:macro name="chenille" params="nom y_signe">
+    <link name="${nom}_chenille">
       <visual>
         <geometry>
           <cylinder radius="${rayon_roue}" length="${largeur_roue}"/>
         </geometry>
-        <origin xyz="0 0 ${-z_folle}" rpy="${pi/2} 0 0"/>
+        <origin xyz="0 0 0" rpy="${pi/2} 0 0"/>
         <material name="noir"/>
       </visual>
@@ -39,5 +39,5 @@
           <cylinder radius="${rayon_roue}" length="${largeur_roue}"/>
         </geometry>
-        <origin xyz="-${empattement_arriere} 0 0" rpy="${pi/2} 0 0"/>
+        <origin xyz="-${empattement_arriere} 0 ${z_folle}" rpy="${pi/2} 0 0"/>
         <material name="argent"/>
       </visual>
@@ -46,5 +46,5 @@
           <cylinder radius="${rayon_roue}" length="${largeur_roue}"/>
         </geometry>
-        <origin xyz="${empattement_avant} 0 0" rpy="${pi/2} 0 0"/>
+        <origin xyz="${empattement_avant} 0 ${z_folle}" rpy="${pi/2} 0 0"/>
         <material name="argent"/>
       </visual>
@@ -53,5 +53,5 @@
           <box size="0.1012 ${largeur_roue} ${2*rayon_roue}"/>
         </geometry>
-        <origin xyz="-0.040 0 ${-z_folle/2}" rpy="0 2.4826 0"/>
+        <origin xyz="-0.040 0 ${z_folle/2}" rpy="0 2.4826 0"/>
         <material name="orange"/>
       </visual>
@@ -60,5 +60,5 @@
           <box size="0.1422 ${largeur_roue} ${2*rayon_roue}"/>
         </geometry>
-        <origin xyz="0.064 0 ${-z_folle/2}" rpy="0 0.4512 0"/>
+        <origin xyz="0.064 0 ${z_folle/2}" rpy="0 0.4512 0"/>
         <material name="noir"/>
       </visual>
@@ -67,7 +67,18 @@
           <box size="0.208 ${largeur_roue} ${2*rayon_roue}"/>
         </geometry>
-        <origin xyz="0.024 0 0" rpy="0 0 0"/>
+        <origin xyz="0.024 0 ${z_folle}" rpy="0 0 0"/>
         <material name="noir"/>
       </visual>
+    </link>
+    <joint name="${nom}_chenille_joint" type="fixed">
+      <parent link="base_link"/>
+      <child  link="${nom}_chenille"/>
+      <origin xyz="0 ${y_signe * y_roue} 0" rpy="0 0 0"/>
+    </joint>
+  </xacro:macro>
+  <!-- Macro de la roue fonctionnelle : invisible, tourne réellement autour de -->
+  <!-- l'axe Y, contact au sol via une collision sphérique ponctuelle -->
+  <xacro:macro name="roue" params="nom y_signe">
+    <link name="${nom}_wheel">
       <collision>
         <geometry>
@@ -88,5 +99,7 @@
     </joint>
   </xacro:macro>
-  <xacro:roue nom="left"  y_signe=" 1"/>
-  <xacro:roue nom="right" y_signe="-1"/>
+  <xacro:chenille nom="left"  y_signe=" 1"/>
+  <xacro:roue     nom="left"  y_signe=" 1"/>
+  <xacro:chenille nom="right" y_signe="-1"/>
+  <xacro:roue     nom="right" y_signe="-1"/>
 </robot>

Commit message: Phase 5 : collision sur le lien chenille (points d'appui avant/arrière), corrige l'instabilité de tangage au spawn

File: src/robot_devastator_description/urdf/roues.xacro (robot description, xacro)
@@ -41,5 +41,5 @@
         </geometry>
         <origin xyz="-${empattement_arriere} 0 ${z_folle}" rpy="${pi/2} 0 0"/>
-        <material name="argent"/>
+        <material name="noir"/>
       </visual>
       <visual>
@@ -48,5 +48,5 @@
         </geometry>
         <origin xyz="${empattement_avant} 0 ${z_folle}" rpy="${pi/2} 0 0"/>
-        <material name="argent"/>
+        <material name="noir"/>
       </visual>
       <visual>
@@ -55,5 +55,5 @@
         </geometry>
         <origin xyz="-0.040 0 ${z_folle/2}" rpy="0 2.4826 0"/>
-        <material name="orange"/>
+        <material name="noir"/>
       </visual>
       <visual>
@@ -71,4 +71,16 @@
         <material name="noir"/>
       </visual>
+      <collision>
+        <geometry>
+          <sphere radius="${rayon_roue}"/>
+        </geometry>
+        <origin xyz="-${empattement_arriere} 0 ${z_folle}" rpy="0 0 0"/>
+      </collision>
+      <collision>
+        <geometry>
+          <sphere radius="${rayon_roue}"/>
+        </geometry>
+        <origin xyz="${empattement_avant} 0 ${z_folle}" rpy="0 0 0"/>
+      </collision>
     </link>
     <joint name="${nom}_chenille_joint" type="fixed">

Commit message: Maj documentation et paramètres

File: src/robot_devastator_description/urdf/roues.xacro (robot description, xacro)
@@ -4,6 +4,6 @@
   <xacro:property name="rayon_roue"   value="0.01966"/>
   <xacro:property name="largeur_roue" value="0.040"/>
-  <!-- Demi-entraxe : chaque roue est à ±0.100 m de base_link -->
-  <xacro:property name="y_roue"       value="0.100"/>
+  <!-- Demi-entraxe : chaque roue est à ±0.985 m de base_link -->
+  <xacro:property name="y_roue"       value="0.985"/>
   <!-- Empattement d'une chenille : distances horizontales depuis le moyeu moteur -->
   <xacro:property name="empattement_arriere" value="0.080"/>
