Commit message: Corrections entraxe Gazebo

File: src/robot_devastator_description/urdf/devastator_gazebo.xacro (robot description, xacro)
@@ -13,5 +13,5 @@
       <left_joint>left_wheel_joint</left_joint>
       <right_joint>right_wheel_joint</right_joint>
-      <wheel_separation>0.200</wheel_separation>
+      <wheel_separation>0.196</wheel_separation>
       <wheel_radius>0.01966</wheel_radius>
       <frame_id>odom</frame_id>

File: src/robot_devastator_description/urdf/roues.xacro (robot description, xacro)
@@ -4,6 +4,6 @@
   <xacro:property name="rayon_roue"   value="0.01966"/>
   <xacro:property name="largeur_roue" value="0.040"/>
-  <!-- Demi-entraxe : chaque roue est à ±0.985 m de base_link -->
-  <xacro:property name="y_roue"       value="0.985"/>
+  <!-- Demi-entraxe : chaque roue est à ±0.098 m de base_link -->
+  <xacro:property name="y_roue"       value="0.098"/>
   <!-- Empattement d'une chenille : distances horizontales depuis le moyeu moteur -->
   <xacro:property name="empattement_arriere" value="0.080"/>
