Commit message: Modélisation et validation du robot (URDF/Xacro + TF + RViz)

File: src/robot_devastator_description/urdf/capteurs.xacro (robot description, xacro)
@@ -2,15 +2,17 @@
 <robot xmlns:xacro="http://www.ros.org/wiki/xacro">
   <!-- Position des capteurs (en mètres, relatifs à base_link) -->
-  <!-- sonar_z = 14.8 cm - 8.2 cm = 6.6 cm -->
+  <!-- Empilement : sommet châssis (12,0 cm) → tourelle → sonar -->
+  <!-- sonar_z = sommet tourelle (14,0 cm) + moitié hauteur sonar (1,5 cm) - base_link_hauteur_sol -->
   <xacro:property name="sonar_x"      value="0.100"/>
-  <xacro:property name="sonar_z"      value="0.066"/>
-  <!-- tourelle_z = 12.0 cm - 8.2 cm = 3.8 cm -->
-  <xacro:property name="tourelle_x"   value="0.000"/>
-  <xacro:property name="tourelle_z"   value="0.038"/>
+  <xacro:property name="sonar_z"      value="0.073"/>
+  <!-- tourelle_z = sommet châssis (12,0 cm) + moitié hauteur tourelle (1,0 cm) - base_link_hauteur_sol -->
+  <xacro:property name="tourelle_x"   value="0.0845"/>
+  <xacro:property name="tourelle_z"   value="0.048"/>
   <!-- Sonar HC-SR04 : petite boîte bleue à l'avant -->
+  <!-- Dimensions : 40 mm x 56 mm x 30 mm (p x l x h) -->
   <link name="sonar_link">
     <visual>
       <geometry>
-        <box size="0.040 0.020 0.020"/>
+        <box size="0.040 0.056 0.030"/>
       </geometry>
       <material name="bleu">
@@ -25,11 +27,12 @@
   </joint>
   <!-- Tourelle servo : petite boîte rouge au centre -->
+  <!-- Dimensions : 53 mm x 20 mm x 20 mm (p x l x h) -->
   <link name="tourelle_link">
     <visual>
       <geometry>
-        <box size="0.050 0.050 0.030"/>
+        <box size="0.053 0.020 0.020"/>
       </geometry>
-      <material name="rouge">
-        <color rgba="1.0 0.0 0.0 1.0"/>
+      <material name="bleu-pale">
+        <color rgba="0.0 0.5 1.0 1.0"/>
       </material>
     </visual>

File: src/robot_devastator_description/urdf/corps.xacro (robot description, xacro)
@@ -4,6 +4,7 @@
   <xacro:property name="chassis_longueur"       value="0.230"/>
   <xacro:property name="chassis_largeur"        value="0.230"/>
-  <xacro:property name="chassis_hauteur"        value="0.120"/>
+  <xacro:property name="chassis_hauteur"        value="0.098"/>
   <xacro:property name="base_link_hauteur_sol"  value="0.082"/>
+  <xacro:property name="chassis_z_offset"       value="-0.011"/>
   <!-- Repère sol — aucune géométrie visuelle -->
   <link name="base_footprint"/>
@@ -20,6 +21,7 @@
         <box size="${chassis_longueur} ${chassis_largeur} ${chassis_hauteur}"/>
       </geometry>
+      <origin xyz="0 0 ${chassis_z_offset}" rpy="0 0 0"/>
       <material name="gris">
-        <color rgba="1.0 0.0 0.0 1.0"/>
+        <color rgba="0.8 0.8 0.8 1.0"/>
       </material>
     </visual>
@@ -28,4 +30,5 @@
         <box size="${chassis_longueur} ${chassis_largeur} ${chassis_hauteur}"/>
       </geometry>
+      <origin xyz="0 0 ${chassis_z_offset}" rpy="0 0 0"/>
     </collision>
     <inertial>

File: src/robot_devastator_description/urdf/roues.xacro (robot description, xacro)
@@ -6,6 +6,24 @@
   <!-- Demi-entraxe : chaque roue est à ±0.100 m de base_link -->
   <xacro:property name="y_roue"       value="0.100"/>
+  <!-- Empattement d'une chenille : distances horizontales depuis le moyeu moteur -->
+  <xacro:property name="empattement_arriere" value="0.080"/>
+  <xacro:property name="empattement_avant"   value="0.128"/>
+  <!-- Roues folles : même rayon que la roue menante (39,32 mm de diamètre) -->
+  <!-- Centre à 20 mm du sol → décalage local = 0,020 - base_link_hauteur_sol (0,082) = -0,062 m -->
+  <xacro:property name="z_folle" value="-0.062"/>
+  <!-- Matériaux des roues : définis une seule fois, référencés par nom ensuite -->
+  <material name="argent">
+    <color rgba="0.6 0.6 0.6 1.0"/>
+  </material>
+  <material name="orange">
+    <color rgba="1.0 0.5 0.0 1.0"/>
+  </material>
+  <material name="noir">
+    <color rgba="0.1 0.1 0.1 1.0"/>
+  </material>
   <!-- Macro réutilisable pour une roue -->
-  <!-- La rotation de π/2 autour de X oriente le cylindre sur l'axe Y -->
+  <!-- La rotation de π/2 autour de X oriente les cylindres sur l'axe Y -->
+  <!-- La géométrie visuelle forme une chenille triangulaire : roue menante + 2 roues -->
+  <!-- folles, reliées par 3 boîtes formant le contour (dont le brin horizontal au sol) -->
   <xacro:macro name="roue" params="nom y_signe">
     <link name="${nom}_wheel">
@@ -15,13 +33,46 @@
         </geometry>
         <origin xyz="0 0 0" rpy="${pi/2} 0 0"/>
-        <material name="noir">
-          <color rgba="0.1 0.1 0.1 1.0"/>
-        </material>
+        <material name="noir"/>
+      </visual>
+      <visual>
+        <geometry>
+          <cylinder radius="${rayon_roue}" length="${largeur_roue}"/>
+        </geometry>
+        <origin xyz="-${empattement_arriere} 0 ${z_folle}" rpy="${pi/2} 0 0"/>
+        <material name="argent"/>
+      </visual>
+      <visual>
+        <geometry>
+          <cylinder radius="${rayon_roue}" length="${largeur_roue}"/>
+        </geometry>
+        <origin xyz="${empattement_avant} 0 ${z_folle}" rpy="${pi/2} 0 0"/>
+        <material name="argent"/>
+      </visual>
+      <visual>
+        <geometry>
+          <box size="0.1012 ${largeur_roue} ${2*rayon_roue}"/>
+        </geometry>
+        <origin xyz="-0.040 0 ${z_folle/2}" rpy="0 2.4826 0"/>
+        <material name="orange"/>
+      </visual>
+      <visual>
+        <geometry>
+          <box size="0.1422 ${largeur_roue} ${2*rayon_roue}"/>
+        </geometry>
+        <origin xyz="0.064 0 ${z_folle/2}" rpy="0 0.4512 0"/>
+        <material name="noir"/>
+      </visual>
+      <visual>
+        <geometry>
+          <box size="0.208 ${largeur_roue} ${2*rayon_roue}"/>
+        </geometry>
+        <origin xyz="0.024 0 ${z_folle}" rpy="0 0 0"/>
+        <material name="noir"/>
       </visual>
       <collision>
         <geometry>
-          <cylinder radius="${rayon_roue}" length="${largeur_roue}"/>
+          <box size="${empattement_arriere+empattement_avant+2*rayon_roue} ${largeur_roue} ${2*rayon_roue}"/>
         </geometry>
-        <origin xyz="0 0 0" rpy="${pi/2} 0 0"/>
+        <origin xyz="${(empattement_avant-empattement_arriere)/2} 0 ${z_folle}" rpy="0 0 0"/>
       </collision>
       <inertial>

Commit message: maj URDF pour ajouter la masse du chassis et des roues ainsi que d'ajouter le pivotement pour sonar_joint

File: src/robot_devastator_description/urdf/capteurs.xacro (robot description, xacro)
@@ -21,8 +21,10 @@
     </visual>
   </link>
-  <joint name="sonar_joint" type="fixed">
+  <joint name="sonar_joint" type="revolute">
     <parent link="base_link"/>
     <child  link="sonar_link"/>
     <origin xyz="${sonar_x} 0 ${sonar_z}" rpy="0 0 0"/>
+    <axis xyz="0 0 1"/>
+    <limit effort="100" velocity="100" lower="-0.78539" upper="0.78539"/>
   </joint>
   <!-- Tourelle servo : petite boîte rouge au centre -->

File: src/robot_devastator_description/urdf/corps.xacro (robot description, xacro)
@@ -7,4 +7,12 @@
   <xacro:property name="base_link_hauteur_sol"  value="0.082"/>
   <xacro:property name="chassis_z_offset"       value="-0.011"/>
+  <xacro:property name="masse_chassis"          value="1.9"/>
+  <!-- Matériaux : définis une seule fois, référencés par nom ensuite -->
+  <material name="bleu_fonce">
+    <color rgba="0 0 0.3 1.0"/>
+  </material>
+  <material name="gris">
+    <color rgba="0.8 0.8 0.8 1.0"/>
+  </material>
   <!-- Repère sol — aucune géométrie visuelle -->
   <link name="base_footprint"/>
@@ -22,7 +30,5 @@
       </geometry>
       <origin xyz="0 0 ${chassis_z_offset}" rpy="0 0 0"/>
-      <material name="gris">
-        <color rgba="0.8 0.8 0.8 1.0"/>
-      </material>
+      <material name="bleu_fonce"/>
     </visual>
     <collision>
@@ -33,6 +39,10 @@
     </collision>
     <inertial>
-      <mass value="1.0"/>
-      <inertia ixx="0.01" ixy="0" ixz="0" iyy="0.01" iyz="0" izz="0.01"/>
+      <mass value="${masse_chassis}"/>
+      <inertia
+        ixx="${masse_chassis*(chassis_largeur*chassis_largeur+chassis_hauteur*chassis_hauteur)/12}"
+        iyy="${masse_chassis*(chassis_longueur*chassis_longueur+chassis_hauteur*chassis_hauteur)/12}"
+        izz="${masse_chassis*(chassis_longueur*chassis_longueur+chassis_largeur*chassis_largeur)/12}"
+        ixy="0" ixz="0" iyz="0"/>
     </inertial>
   </link>

File: src/robot_devastator_description/urdf/roues.xacro (robot description, xacro)
@@ -9,8 +9,9 @@
   <xacro:property name="empattement_arriere" value="0.080"/>
   <xacro:property name="empattement_avant"   value="0.128"/>
+  <xacro:property name="masse_roue" value="0.1"/>
   <!-- Roues folles : même rayon que la roue menante (39,32 mm de diamètre) -->
   <!-- Centre à 20 mm du sol → décalage local = 0,020 - base_link_hauteur_sol (0,082) = -0,062 m -->
   <xacro:property name="z_folle" value="-0.062"/>
-  <!-- Matériaux des roues : définis une seule fois, référencés par nom ensuite -->
+  <!-- Matériaux : définis une seule fois, référencés par nom ensuite -->
   <material name="argent">
     <color rgba="0.6 0.6 0.6 1.0"/>
@@ -88,6 +89,10 @@
       </collision>
       <inertial>
-        <mass value="0.1"/>
-        <inertia ixx="0.001" ixy="0" ixz="0" iyy="0.001" iyz="0" izz="0.001"/>
+        <mass value="${masse_roue}"/>
+        <inertia
+          ixx="${masse_roue*(3*rayon_roue*rayon_roue+largeur_roue*largeur_roue)/12}"
+          iyy="${masse_roue*rayon_roue*rayon_roue/2}"
+          izz="${masse_roue*(3*rayon_roue*rayon_roue+largeur_roue*largeur_roue)/12}"
+          ixy="0" ixz="0" iyz="0"/>
       </inertial>
     </link>

Commit message: Phase 5 : inertial et collision réalistes (chassis, roues, sonar) + limite angle sonar ±45°

File: src/robot_devastator_description/urdf/capteurs.xacro (robot description, xacro)
@@ -9,4 +9,12 @@
   <xacro:property name="tourelle_x"   value="0.0845"/>
   <xacro:property name="tourelle_z"   value="0.048"/>
+  <xacro:property name="masse_sonar"  value="0.010"/>
+  <!-- Matériaux : définis une seule fois, référencés par nom ensuite -->
+  <material name="bleu">
+    <color rgba="0.0 0.0 1.0 1.0"/>
+  </material>
+  <material name="bleu_pale">
+    <color rgba="0.0 0.5 1.0 1.0"/>
+  </material>
   <!-- Sonar HC-SR04 : petite boîte bleue à l'avant -->
   <!-- Dimensions : 40 mm x 56 mm x 30 mm (p x l x h) -->
@@ -16,8 +24,19 @@
         <box size="0.040 0.056 0.030"/>
       </geometry>
-      <material name="bleu">
-        <color rgba="0.0 0.0 1.0 1.0"/>
-      </material>
+      <material name="bleu"/>
     </visual>
+    <collision>
+      <geometry>
+        <box size="0.040 0.056 0.030"/>
+      </geometry>
+    </collision>
+    <inertial>
+      <mass value="${masse_sonar}"/>
+      <inertia
+        ixx="${masse_sonar*(0.056*0.056+0.030*0.030)/12}"
+        iyy="${masse_sonar*(0.040*0.040+0.030*0.030)/12}"
+        izz="${masse_sonar*(0.040*0.040+0.056*0.056)/12}"
+        ixy="0" ixz="0" iyz="0"/>
+    </inertial>
   </link>
   <joint name="sonar_joint" type="revolute">
@@ -35,7 +54,5 @@
         <box size="0.053 0.020 0.020"/>
       </geometry>
-      <material name="bleu-pale">
-        <color rgba="0.0 0.5 1.0 1.0"/>
-      </material>
+      <material name="bleu_pale"/>
     </visual>
   </link>

Commit message: Maj URDF pour ajout RPLiDAR

File: src/robot_devastator_description/urdf/capteurs.xacro (robot description, xacro)
@@ -9,4 +9,8 @@
   <xacro:property name="tourelle_x"   value="0.0845"/>
   <xacro:property name="tourelle_z"   value="0.048"/>
+  <!-- Position mesurée du RPLIDAR A1M8, relative à base_link -->
+  <xacro:property name="laser_x"      value="-0.075"/>
+  <xacro:property name="laser_y"      value="-0.010"/>
+  <xacro:property name="laser_z"      value="0.101"/>
   <xacro:property name="masse_sonar"  value="0.010"/>
   <!-- Matériaux : définis une seule fois, référencés par nom ensuite -->
@@ -17,4 +21,5 @@
     <color rgba="0.0 0.5 1.0 1.0"/>
   </material>
+  <!-- "gris" est déjà défini dans corps.xacro : réutilisé tel quel pour laser_link -->
   <!-- Sonar HC-SR04 : petite boîte bleue à l'avant -->
   <!-- Dimensions : 40 mm x 56 mm x 30 mm (p x l x h) -->
@@ -62,3 +67,19 @@
     <origin xyz="${tourelle_x} 0 ${tourelle_z}" rpy="0 0 0"/>
   </joint>
+  <!-- RPLIDAR A1M8 : cylindre gris sur le dessus du châssis -->
+  <!-- Dimensions approximatives (pas de fiche technique précise sous la main) :
+       rayon 38 mm (diamètre ~76 mm), hauteur 40 mm -->
+  <link name="laser_link">
+    <visual>
+      <geometry>
+        <cylinder radius="0.038" length="0.040"/>
+      </geometry>
+      <material name="gris"/>
+    </visual>
+  </link>
+  <joint name="laser_joint" type="fixed">
+    <parent link="base_link"/>
+    <child  link="laser_link"/>
+    <origin xyz="${laser_x} ${laser_y} ${laser_z}" rpy="0 0 0"/>
+  </joint>
 </robot>

Commit message: Correction pour Gazebo

File: src/robot_devastator_description/urdf/capteurs.xacro (robot description, xacro)
@@ -10,7 +10,37 @@
   <xacro:property name="tourelle_z"   value="0.048"/>
   <!-- Position mesurée du RPLIDAR A1M8, relative à base_link -->
-  <xacro:property name="laser_x"      value="-0.075"/>
-  <xacro:property name="laser_y"      value="-0.010"/>
-  <xacro:property name="laser_z"      value="0.101"/>
+  <xacro:property name="laser_x"      value="-0.080"/>
+  <xacro:property name="laser_y"      value="-0.015"/>
+  <xacro:property name="laser_z"      value="0.150"/>
+  <!-- Empilement du support lidar, sur le dessus du châssis, à l'arrière (X négatif) -->
+  <!-- Dimensions des boîtes de support (en mètres) : L x P x H -->
+  <xacro:property name="plateforme_lidar_longueur" value="0.130"/>
+  <xacro:property name="plateforme_lidar_largeur"  value="0.160"/>
+  <xacro:property name="plateforme_lidar_hauteur"  value="0.070"/>
+  <!-- plateforme_lidar_x : fond aligné sur le fond (arrière) du châssis, comme le RPLIDAR
+       fond châssis = -chassis_longueur/2 = -0.115 ; centre = -0.115 + largeur/2, car le
+       visual/collision est tourné de 90° en Z (voir plateforme_lidar_link) : la dimension
+       effective en X devient plateforme_lidar_largeur, pas plateforme_lidar_longueur -->
+  <xacro:property name="plateforme_lidar_x" value="-0.035"/>
+  <!-- plateforme_lidar_z = sommet châssis (12,0 cm) + moitié hauteur plateforme (3,5 cm)
+       - base_link_hauteur_sol -->
+  <xacro:property name="plateforme_lidar_z" value="0.073"/>
+  <xacro:property name="masse_plateforme_lidar" value="0.030"/>
+  <xacro:property name="base_lidar_longueur" value="0.070"/>
+  <xacro:property name="base_lidar_largeur"  value="0.100"/>
+  <xacro:property name="base_lidar_hauteur"  value="0.030"/>
+  <!-- base_lidar_x : fond aligné sur le fond (arrière) du châssis, comme plateforme_lidar_link
+       fond châssis = -0.115 ; centre = -0.115 + largeur/2, car le visual/collision est tourné
+       de 90° en Z (voir base_lidar_link) : la dimension effective en X devient
+       base_lidar_largeur, pas base_lidar_longueur -->
+  <xacro:property name="base_lidar_x" value="-0.065"/>
+  <!-- base_lidar_z = sommet plateforme_lidar (19,0 cm) + moitié hauteur base (1,5 cm)
+       - base_link_hauteur_sol -->
+  <xacro:property name="base_lidar_z" value="0.123"/>
+  <xacro:property name="masse_base_lidar" value="0.010"/>
+  <!-- Dimensions du RPLIDAR A1M8, mesures directes sur le robot réel -->
+  <xacro:property name="laser_rayon"    value="0.035"/>
+  <xacro:property name="laser_longueur" value="0.024"/>
+  <xacro:property name="masse_laser"    value="0.190"/>
   <xacro:property name="masse_sonar"  value="0.010"/>
   <!-- Matériaux : définis une seule fois, référencés par nom ensuite -->
@@ -21,5 +51,6 @@
     <color rgba="0.0 0.5 1.0 1.0"/>
   </material>
-  <!-- "gris" est déjà défini dans corps.xacro : réutilisé tel quel pour laser_link -->
+  <!-- "gris" et "bleu_fonce" sont déjà définis dans corps.xacro, "noir" dans roues.xacro :
+       réutilisés tels quels -->
   <!-- Sonar HC-SR04 : petite boîte bleue à l'avant -->
   <!-- Dimensions : 40 mm x 56 mm x 30 mm (p x l x h) -->
@@ -68,13 +99,26 @@
   </joint>
   <!-- RPLIDAR A1M8 : cylindre gris sur le dessus du châssis -->
-  <!-- Dimensions approximatives (pas de fiche technique précise sous la main) :
-       rayon 38 mm (diamètre ~76 mm), hauteur 40 mm -->
+  <!-- Dimensions mesurées directement sur le robot réel : rayon 35 mm (diamètre 70 mm),
+       hauteur 24 mm -->
   <link name="laser_link">
     <visual>
       <geometry>
-        <cylinder radius="0.038" length="0.040"/>
+        <cylinder radius="${laser_rayon}" length="${laser_longueur}"/>
       </geometry>
-      <material name="gris"/>
+      <material name="noir"/>
     </visual>
+    <collision>
+      <geometry>
+        <cylinder radius="${laser_rayon}" length="${laser_longueur}"/>
+      </geometry>
+    </collision>
+    <inertial>
+      <mass value="${masse_laser}"/>
+      <inertia
+        ixx="${masse_laser*(3*laser_rayon*laser_rayon+laser_longueur*laser_longueur)/12}"
+        iyy="${masse_laser*(3*laser_rayon*laser_rayon+laser_longueur*laser_longueur)/12}"
+        izz="${masse_laser*laser_rayon*laser_rayon/2}"
+        ixy="0" ixz="0" iyz="0"/>
+    </inertial>
   </link>
   <joint name="laser_joint" type="fixed">
@@ -83,3 +127,69 @@
     <origin xyz="${laser_x} ${laser_y} ${laser_z}" rpy="0 0 0"/>
   </joint>
+  <!-- Plateforme lidar : boîte de support posée sur le dessus du châssis, fond aligné sur
+       l'arrière du châssis (X négatif), centrée en Y -->
+  <!-- Rotation de 90° en Z : plateforme_lidar_longueur/largeur sont définies selon les
+       dimensions physiques mesurées (L en X, P en Y), mais le repère X/Y de la boîte doit être
+       tourné pour correspondre à l'orientation réelle du support sur le châssis -->
+  <link name="plateforme_lidar_link">
+    <visual>
+      <origin xyz="0 0 0" rpy="0 0 1.5708"/>
+      <geometry>
+        <box size="${plateforme_lidar_longueur} ${plateforme_lidar_largeur} ${plateforme_lidar_hauteur}"/>
+      </geometry>
+      <material name="bleu_fonce"/>
+    </visual>
+    <collision>
+      <origin xyz="0 0 0" rpy="0 0 1.5708"/>
+      <geometry>
+        <box size="${plateforme_lidar_longueur} ${plateforme_lidar_largeur} ${plateforme_lidar_hauteur}"/>
+      </geometry>
+    </collision>
+    <!-- Masse non mesurée, valeur symbolique -->
+    <inertial>
+      <mass value="${masse_plateforme_lidar}"/>
+      <inertia
+        ixx="${masse_plateforme_lidar*(plateforme_lidar_largeur*plateforme_lidar_largeur+plateforme_lidar_hauteur*plateforme_lidar_hauteur)/12}"
+        iyy="${masse_plateforme_lidar*(plateforme_lidar_longueur*plateforme_lidar_longueur+plateforme_lidar_hauteur*plateforme_lidar_hauteur)/12}"
+        izz="${masse_plateforme_lidar*(plateforme_lidar_longueur*plateforme_lidar_longueur+plateforme_lidar_largeur*plateforme_lidar_largeur)/12}"
+        ixy="0" ixz="0" iyz="0"/>
+    </inertial>
+  </link>
+  <joint name="plateforme_lidar_joint" type="fixed">
+    <parent link="base_link"/>
+    <child  link="plateforme_lidar_link"/>
+    <origin xyz="${plateforme_lidar_x} 0 ${plateforme_lidar_z}" rpy="0 0 0"/>
+  </joint>
+  <!-- Base lidar : boîte de support posée sur le dessus de plateforme_lidar_link, fond aligné
+       sur l'arrière du châssis comme plateforme_lidar_link, centrée en Y -->
+  <!-- Rotation de 90° en Z : même correctif d'orientation que plateforme_lidar_link -->
+  <link name="base_lidar_link">
+    <visual>
+      <origin xyz="0 0 0" rpy="0 0 1.5708"/>
+      <geometry>
+        <box size="${base_lidar_longueur} ${base_lidar_largeur} ${base_lidar_hauteur}"/>
+      </geometry>
+      <material name="bleu_fonce"/>
+    </visual>
+    <collision>
+      <origin xyz="0 0 0" rpy="0 0 1.5708"/>
+      <geometry>
+        <box size="${base_lidar_longueur} ${base_lidar_largeur} ${base_lidar_hauteur}"/>
+      </geometry>
+    </collision>
+    <!-- Masse non mesurée, valeur symbolique -->
+    <inertial>
+      <mass value="${masse_base_lidar}"/>
+      <inertia
+        ixx="${masse_base_lidar*(base_lidar_largeur*base_lidar_largeur+base_lidar_hauteur*base_lidar_hauteur)/12}"
+        iyy="${masse_base_lidar*(base_lidar_longueur*base_lidar_longueur+base_lidar_hauteur*base_lidar_hauteur)/12}"
+        izz="${masse_base_lidar*(base_lidar_longueur*base_lidar_longueur+base_lidar_largeur*base_lidar_largeur)/12}"
+        ixy="0" ixz="0" iyz="0"/>
+    </inertial>
+  </link>
+  <joint name="base_lidar_joint" type="fixed">
+    <parent link="base_link"/>
+    <child  link="base_lidar_link"/>
+    <origin xyz="${base_lidar_x} 0 ${base_lidar_z}" rpy="0 0 0"/>
+  </joint>
 </robot>

File: src/robot_devastator_description/urdf/devastator_gazebo.xacro (robot description, xacro)
@@ -8,4 +8,26 @@
     <mu1>0.1</mu1>
     <mu2>0.1</mu2>
+  </gazebo>
+  <!-- Couleurs explicites pour Gazebo : capteurs.xacro référence des matériaux déclarés dans
+       d'autres fichiers (bleu_fonce dans corps.xacro, noir dans roues.xacro), ce que la
+       conversion URDF -> SDF de Gazebo Harmonic ne résout pas de façon fiable à travers les
+       fichiers xacro assemblés. RViz n'a pas ce problème (table de matériaux globale). -->
+  <gazebo reference="plateforme_lidar_link">
+    <material>
+      <ambient>0 0 0.3 1.0</ambient>
+      <diffuse>0 0 0.3 1.0</diffuse>
+    </material>
+  </gazebo>
+  <gazebo reference="base_lidar_link">
+    <material>
+      <ambient>0 0 0.3 1.0</ambient>
+      <diffuse>0 0 0.3 1.0</diffuse>
+    </material>
+  </gazebo>
+  <gazebo reference="laser_link">
+    <material>
+      <ambient>0.1 0.1 0.1 1.0</ambient>
+      <diffuse>0.1 0.1 0.1 1.0</diffuse>
+    </material>
   </gazebo>
   <gazebo>
@@ -30,4 +52,12 @@
       <render_engine>ogre2</render_engine>
     </plugin>
+  </gazebo>
+  <!-- laser_joint est fixed et relie laser_link à base_link, lui-même fusionné dans
+       base_footprint via base_footprint_joint (fixed). Sans cette directive, sdformat
+       fusionne récursivement laser_link jusque dans base_footprint lors de la conversion
+       URDF -> SDF : le lien laser_link disparaît, et le capteur ci-dessous ne trouve plus
+       sa référence (avertissement Gazebo, /scan ne publie rien). -->
+  <gazebo reference="laser_joint">
+    <disableFixedJointLumping>true</disableFixedJointLumping>
   </gazebo>
   <!-- Lidar simulé, calqué sur le RPLIDAR A1M8 réel (laser_link, voir capteurs.xacro).
